Commit message: add arx5 agent

File: mani_skill2_real2sim/assets/descriptions/arx5_description/arx5_description_isaac.urdf (robot description, URDF)
Before this commit: robot arx5_description, 56 links, 55 joints
Joints:
- joint fl_castor_wheel: type continuous -> fixed
- joint fl_joint7: type prismatic -> revolute
- joint fl_joint8: type prismatic -> revolute
- joint fl_wheel: type continuous -> fixed
- joint fr_castor_wheel: type continuous -> fixed
- joint fr_joint7: type prismatic -> revolute
- joint fr_joint8: type prismatic -> revolute
- joint fr_wheel: type continuous -> fixed
- joint left_wheel: type continuous -> fixed
- joint lr_joint1: type revolute -> fixed
- joint lr_joint2: type revolute -> fixed
- joint lr_joint3: type revolute -> fixed
- joint lr_joint4: type revolute -> fixed
- joint lr_joint5: type revolute -> fixed
- joint lr_joint6: type revolute -> fixed
- joint lr_joint7: type prismatic -> fixed
- joint lr_joint8: type prismatic -> fixed
- joint right_wheel: type continuous -> fixed
- joint rl_castor_wheel: type continuous -> fixed
- joint rl_wheel: type continuous -> fixed
- joint rr_castor_wheel: type continuous -> fixed
- joint rr_joint1: type revolute -> fixed
- joint rr_joint2: type revolute -> fixed
- joint rr_joint3: type revolute -> fixed
- joint rr_joint4: type revolute -> fixed
- joint rr_joint5: type revolute -> fixed
- joint rr_joint6: type revolute -> fixed
- joint rr_joint7: type prismatic -> fixed
- joint rr_joint8: type prismatic -> fixed
- joint rr_wheel: type continuous -> fixed
